Commit message: changes to hes probe urdf

File: urdf/hes_probe.urdf.xacro (robot description, xacro)
@@ -17,4 +17,8 @@
         <link name="${probe_name}_lens" />
         <link name="${probe_name}_standoff" />
+        <link name="${probe_name}_mount_point_1"/>
+        <link name="${probe_name}_mount_point_2"/>
+        <link name="${probe_name}_mount_point_3"/>
+        <link name="${probe_name}_mount_point_4"/>
         <link name="${probe_name}_center">
             <visual>
@@ -48,15 +52,35 @@
             <parent link="${probe_name}_base_link"/>
             <child link="${probe_name}_center"/>
-            <origin xyz="0 0 0" rpy="0 0 0" />
+            <origin xyz="0 0 0.05" rpy="0 0 0" />
         </joint>
         <joint name="${probe_name}_center_lens" type="fixed">
             <parent link="${probe_name}_center"/>
             <child link="${probe_name}_lens"/>
-            <origin xyz="0 0 0" rpy="${-pi/2} 0 0" />
+            <origin xyz="0 0.1 0" rpy="${-pi/2} 0 0" />
         </joint>
         <joint name="${probe_name}_lens_standoff" type="fixed">
             <parent link="${probe_name}_lens"/>
             <child link="${probe_name}_standoff"/>
-            <origin xyz="0 0 0" rpy="0 0 0" />
+            <origin xyz="0 0 1" rpy="0 0 0" />
+        </joint>
+        <joint name="${probe_name}_mount_point_1_joint" type="fixed">
+            <parent link="${probe_name}_base_link"/>
+            <child link="${probe_name}_mount_point_1"/>
+            <origin xyz="0.0176775 0.0176775 0" rpy="0 0 0" />
+        </joint>
+        <joint name="${probe_name}_mount_point_2_joint" type="fixed">
+            <parent link="${probe_name}_base_link"/>
+            <child link="${probe_name}_mount_point_2"/>
+            <origin xyz="-0.0176775 0.0176775 0" rpy="0 0 0" />
+        </joint>
+        <joint name="${probe_name}_mount_point_3_joint" type="fixed">
+            <parent link="${probe_name}_base_link"/>
+            <child link="${probe_name}_mount_point_3"/>
+            <origin xyz="0.0176775 -0.0176775 0" rpy="0 0 0" />
+        </joint>
+        <joint name="${probe_name}_mount_point_4_joint" type="fixed">
+            <parent link="${probe_name}_base_link"/>
+            <child link="${probe_name}_mount_point_4"/>
+            <origin xyz="-0.0176775 -0.0176775 0" rpy="0 0 0" />
         </joint>
     </xacro:macro>

Commit message: update urdf mesh

File: urdf/hes_probe.urdf.xacro (robot description, xacro)
@@ -6,6 +6,6 @@
     <xacro:macro name="isi_hes_probe" params="probe_name:=hes_probe en_mesh:=false">
         <xacro:property name="mesh_file" value="package://isi_hes_base/mesh/hes_probe.stl"/>
-        <xacro:property name="mesh_offset_xyz" value="0 0 0"/>
-        <xacro:property name="mesh_offset_rpy" value="0 0 0"/>
+        <xacro:property name="mesh_offset_xyz" value="0 0.081 0"/>
+        <xacro:property name="mesh_offset_rpy" value="${pi/2} 0 ${pi}"/>
         <xacro:property name="box_offset_xyz" value="0 0 0"/>
         <xacro:property name="box_offset_rpy" value="0 0 0"/>
@@ -17,4 +17,5 @@
         <link name="${probe_name}_lens" />
         <link name="${probe_name}_standoff" />
+        <link name="${probe_name}_camera_mount" />
         <link name="${probe_name}_mount_point_1"/>
         <link name="${probe_name}_mount_point_2"/>
@@ -49,13 +50,18 @@
             <origin xyz="0 0 0" rpy="0 0 0" />
         </joint>
+        <joint name="${probe_name}_base_camera_mount" type="fixed">
+            <parent link="${probe_name}_base_link"/>
+            <child link="${probe_name}_camera_mount"/>
+            <origin xyz="0 0.245 0" rpy="0 0 0" />
+        </joint>
         <joint name="${probe_name}_base_center" type="fixed">
             <parent link="${probe_name}_base_link"/>
             <child link="${probe_name}_center"/>
-            <origin xyz="0 0 0.05" rpy="0 0 0" />
+            <origin xyz="0 0 0.068" rpy="0 0 0" />
         </joint>
         <joint name="${probe_name}_center_lens" type="fixed">
             <parent link="${probe_name}_center"/>
             <child link="${probe_name}_lens"/>
-            <origin xyz="0 0.1 0" rpy="${-pi/2} 0 0" />
+            <origin xyz="0 0.245 0" rpy="${-pi/2} 0 0" />
         </joint>
         <joint name="${probe_name}_lens_standoff" type="fixed">

File: urdf/hes_probe_scene.urdf.xacro (robot description, xacro)
@@ -6,4 +6,11 @@
     xmlns:xacro="http://ros.org/wiki/xacro">
     <xacro:include filename="$(find isi_hes_base)/urdf/hes_probe.urdf.xacro"/>
-    <xacro:isi_hes_probe en_mesh="true"/>
+    <xacro:include filename="$(find i3dr_deimos)/urdf/deimos.urdf.xacro"/>
+    <xacro:isi_hes_probe probe_name="hes_probe" en_mesh="true"/>
+    <xacro:deimos_camera camera_name="deimos" en_mesh="true"/>
+    <joint name="hes_probe_camera_mount" type="fixed">
+        <parent link="hes_probe_camera_mount"/>
+        <child link="deimos_base_link"/>
+        <origin xyz="0 0 0" rpy="0 0 0" />
+    </joint>
 </robot>
